File: odrive_aux_interface.kicad_pcb (KiCad board)
At the start: 2 copper layers, 46.4 x 83.8 mm, 42 parts, among them J1 Conn_01x20_Male, J10 Conn_01x03, J11 Conn_01x03, J12 Conn_01x06, J13 Conn_01x02, J14 Conn_01x03, J2 Conn_01x03, J3 Conn_01x03, J4 Conn_01x03, J5 Conn_01x03, J6 Conn_01x04, J7 Conn_01x06, J8 Conn_01x03, J9 Conn_01x03, U1 EL814

Commit message: Update to v1.2, add gerbers.
Parts:
- removed the J12 at (125.7, 146.7)
- removed the J13 at (138.4, 163.8)
- removed the J6 at (125.7, 113.7)
- removed TP10, TP11, TP12, TP13, TP14, TP15, TP16, TP17, TP2, TP3, TP6, TP7, TP8, TP9: TestPoint, TestPoint:TestPoint_Keystone_5015_Micro-Minature
- added C5: 4000pF NP0, Capacitor_SMD:C_0805_2012Metric, F.Cu at (141.2, 163.8)
- added C6: 4000pF NP0, Capacitor_SMD:C_0805_2012Metric, F.Cu at (148.8, 163.8)
- added C7: 0.1uF, Capacitor_SMD:C_0805_2012Metric, F.Cu at (139.0, 103.5)
- added C8: 0.1uF, Capacitor_SMD:C_0805_2012Metric, F.Cu at (145.0, 163.8)
- added D4: CDSOT23-SM712, digikey-footprints:SOT-23-3, F.Cu at (132.5, 99.0)
- added D5: CDSOT23-SM712, digikey-footprints:SOT-23-3, F.Cu at (133.5, 109.0)
- added J15: Conn_01x05, Connector_JST:JST_XH_B5B-XH-A_1x05_P2.50mm_Vertical, F.Cu at (126.0, 100.0)
- added J16: RJ45_LED_Shielded, Connector_RJ:RJ45_Amphenol_RJHSE538X, F.Cu at (132.8, 164.0)
- added J2: Conn_01x02, Connector_JST:JST_XH_B2B-XH-A_1x02_P2.50mm_Vertical, F.Cu at (126.0, 147.0)
- added J7: Conn_01x02, Connector_JST:JST_XH_B2B-XH-A_1x02_P2.50mm_Vertical, F.Cu at (144.0, 169.0)
- added R10: 750R, Resistor_SMD:R_0805_2012Metric, F.Cu at (136.0, 97.0)
- added R11: 10k, Resistor_SMD:R_0805_2012Metric, F.Cu at (137.2, 151.0)
- added R12: 500R, Resistor_SMD:R_0805_2012Metric, F.Cu at (134.0, 152.5)
- added R13: 500R, Resistor_SMD:R_0805_2012Metric, F.Cu at (129.5, 153.5)
- added R3: 1M, Resistor_SMD:R_0805_2012Metric, F.Cu at (145.0, 161.8)
- added R4: 1M, Resistor_SMD:R_0805_2012Metric, F.Cu at (139.8, 159.2)
- added R5: 750R, Resistor_SMD:R_0805_2012Metric, F.Cu at (137.0, 109.0)
- added R6: 130R, Resistor_SMD:R_0805_2012Metric, F.Cu at (133.5, 112.5)
- added R7: 750R, Resistor_SMD:R_0805_2012Metric, F.Cu at (130.5, 111.0)
- added R8: 750R, Resistor_SMD:R_0805_2012Metric, F.Cu at (132.5, 93.0)
- added R9: 130R, Resistor_SMD:R_0805_2012Metric, F.Cu at (132.5, 95.5)
- added U2: THVD1451D, Package_SO:SOIC-8_3.9x4.9mm_P1.27mm, F.Cu at (133.5, 104.0)
- added U4: UCC2946D, Package_SO:SO-8_3.9x4.9mm_P1.27mm, F.Cu at (145.2, 157.8)
- R2: renamed from R1; value 20k -> 10k
- moved TP4 22.9 mm to (144.5, 150.5)
- moved R1 16.4 mm to (132.2, 148.8), turned to 0 degrees
- moved U1 14.8 mm to (134.5, 142.2)
- moved J13 14.3 mm to (126.0, 116.5)
- moved J12 12.9 mm to (159.5, 161.0), turned to 180 degrees
- moved TP1 6.33 mm to (155.0, 169.5), turned to 90 degrees
- moved J11 2.96 mm to (159.4, 153.2)
- moved R2 2.76 mm to (143.8, 153.8), turned to 180 degrees
- moved J10 2.07 mm to (159.4, 145.2)
- moved J9 0.93 mm to (159.4, 137.5)
- moved J8 0.27 mm to (126.0, 127.6)
- renumbered J9 to J10, J10 to J11, J11 to J12, J14 to J13, J2 to J3, J3 to J4, J4 to J5, J5 to J6, J7 to J8, J8 to J9, R2 to R1
Connections:
- R1 pad 1: Net-(J13-Pad1) -> E1
- R2 pad 1: GPIO_8 -> WDI
- U1 pad 2: Net-(J13-Pad2) -> E2
- U1 pad 3: GPIO_8 -> WDI
Routing:
- net GND: track 226.1 -> 22.6 mm, vias 1 -> 0
- net Net-(D4-Pad1): track 0.00 -> 100.1 mm, vias 0 -> 2
- net 3v3: track 172.9 -> 91.7 mm, vias 1 -> 5
- net Net-(D4-Pad2): track 0.00 -> 79.9 mm
- net Net-(D5-Pad2): track 0.00 -> 79.1 mm, vias 0 -> 2
- net Net-(D5-Pad1): track 0.00 -> 67.3 mm, vias 0 -> 1
- net WDI: track 0.00 -> 37.2 mm, vias 0 -> 2
- net SPI_MISO: track 53.4 -> 17.3 mm, vias 1 -> 0
- net E2: track 0.00 -> 31.5 mm
- net GPIO_6: track 43.3 -> 15.5 mm
- net SPI_MOSI: track 45.4 -> 17.8 mm
- net SPI_SCK: track 44.7 -> 17.4 mm
- net E1: track 0.00 -> 23.9 mm, vias 0 -> 1
- net GPIO_2: track 66.7 -> 87.4 mm, vias 0 -> 4
- net E_SWITCH1: track 0.00 -> 18.6 mm
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- added copper zone on B.Cu, net 3v3
- added copper zone on F.Cu, net GND
Other:
- board text added: "EAUX"
- board text added: "ESWITCH"
- board text added: "Odrive Aux V1.2 CC0 License Love Everyone"
- board text added: "RS-485"
- board text removed: "ESTOP"
- board text removed: "Odrive Aux V1.0 CC0 License Love Everyone"
- board text removed: "SPI_2"
- board text removed: "UART"
